Commit message: tambahan gazebo dalam membuat 3D model mobile robot

File: chapter_2_codes/urdf/diff_wheeled_robot.xacro (robot description, xacro)
@@ -161,3 +161,74 @@
   </gazebo>
 <!-- Caster Back -->
+<!-- Wheel Definitions -->
+  <!-- <wheel fb="front" lr="right" parent="base_link" translateX="posisi x ban terhadap base_link" translateY="posisi y ban terhadap base_link" flipY="kemiringan si ban terhadap base_link, kalau 1 tegak lurus, 2 sejajar, 1.5 miring dia"/> -->
+  <wheel fb="front" lr="right" parent="base_link" translateX="0" translateY="0.5" flipY="1"/>
+  <wheel fb="front" lr="left" parent="base_link" translateX="0" translateY="-0.5" flipY="1"/>
+<!-- ============ SENSORS ============ -->
+  <!-- Hokuyo -->
+  <link name="hokuyo_link">
+    <visual>
+      <origin xyz="0.0 0.0 0.0" rpy="0.0 0.0 0.0"/>
+      <geometry>
+        <box size="${hokuyo_size} ${hokuyo_size} ${hokuyo_size}"/>
+      </geometry>
+      <material name="Blue"/>
+    </visual>
+  </link>
+  <joint name="hokuyo_joint" type="fixed">
+    <origin xyz="${base_radius - hokuyo_size/2} 0.0 ${base_height + hokuyo_size/4}" rpy="0.0 0.0 0.0"/>     <!-- Posisi sensor terhadap base_link -->
+    <parent link="base_link"/>
+    <child link="hokuyo_link"/>
+  </joint>
+  <gazebo reference="hokuyo_link">
+    <material>Gasebo/Blue</material>
+    <turnGravityOff>false</turnGravityOff>
+    <sensor type="ray" name="head_hokuyo_sensor">
+      <pose>${hokuyo_size/2} 0 0 0 0 0</pose>
+      <visualize>false</visualize>
+      <update_rate>40</update_rate>
+      <ray>
+        <scan>
+          <horizontal>
+            <samples>720</samples>
+            <resolution>1</resolution>
+            <min_angle>-1.570796</min_angle>
+            <max_angle>1.570796</max_angle>
+          </horizontal>
+        </scan>
+        <range>
+          <min>0.10</min>
+          <max>10.0</max>
+          <resolution>0.001</resolution>
+        </range>
+      </ray>
+      <plugin name="gazebo_ros_head_hokuyo_controller" filename="libgazebo_ros_laser.so">
+        <topicName>/scan</topicName>
+        <frameName>hokuyo_link</frameName>
+      </plugin>
+    </sensor>
+  </gazebo>
+<!-- ============== Differential drive controller ============== -->
+  <gazebo>
+    <plugin name="differential_drive_controller" filename="libgazebo_ros_diff_drive.so">
+      <rosDebugLevel>Debug</rosDebugLevel>
+      <publishWheelTF>false</publishWheelTF>
+      <robotNamespace>/</robotNamespace>
+      <publishTf>1</publishTf>
+      <publishWheelJointState>false</publishWheelJointState>
+      <alwaysOn>true</alwaysOn>
+      <updateRate>100.0</updateRate>
+      <leftJoint>front_left_wheel_joint</leftJoint>
+      <rightJoint>front_right_wheel_joint</rightJoint>
+      <wheelSeparation>${2*base_radius}</wheelSeparation>
+      <wheelDiameter>${2*wheel_radius}</wheelDiameter>
+      <broadcastTF>1</broadcastTF>
+      <wheelTorque>30</wheelTorque>
+      <wheelAcceleration>1.8</wheelAcceleration>
+      <commandTopic>cmd_vel</commandTopic>
+      <odometryFrame>odom</odometryFrame>
+      <odometryTopic>odom</odometryTopic>
+      <robotBaseFrame>base_footprint</robotBaseFrame>
+    </plugin>
+  </gazebo>
 </robot>

Commit message: tambahin gazebo di file .launch supaya bisa disimulasikan di gazebo

File: chapter_2_codes/urdf/diff_wheeled_robot.xacro (robot description, xacro)
@@ -182,5 +182,5 @@
   </joint>
   <gazebo reference="hokuyo_link">
-    <material>Gasebo/Blue</material>
+    <material>Gazebo/Blue</material>
     <turnGravityOff>false</turnGravityOff>
     <sensor type="ray" name="head_hokuyo_sensor">
